Commit message: Move the ugv_rover sensor frames to the Jetson Orin kit's CAD

File: src/ugv_main/ugv_description/urdf/bases/ugv_rover.xacro (robot description, xacro)
@@ -13,4 +13,9 @@
 <xacro:arg name="add_depth_camera" default="false"/>
 <xacro:property name="add_depth_camera" value="$(arg add_depth_camera)"/>
+<!-- kit: "jetson_orin" (default) places the deck sensors and the pan-tilt as on the
+     UGV Rover PT Jetson Orin ROS2 Kit, measured on Waveshare's STEP model
+     (docs/MODEL_CHANGES.md). "upstream" keeps Waveshare's original values. -->
+<xacro:arg name="kit" default="jetson_orin"/>
+<xacro:property name="kit" value="$(arg kit)"/>
 <xacro:arg name="robot_namespace" default="/" />
 <xacro:arg name="urdf_extras" default="empty.urdf" />
@@ -18,7 +23,22 @@
 <xacro:include filename="$(find ugv_description)/urdf/wheels/rover_wheel.xacro" />
 <xacro:include filename="$(find ugv_description)/urdf/sensors/lidar.xacro" />
+<xacro:if value="${kit == 'upstream'}">
 <xacro:property name="lidar_joint_pose">
   <origin xyz="0.03170 -0.00102 0.04" rpy="0 0 1.5708"/>
 </xacro:property>
+<xacro:property name="oak_joint_pose">
+  <origin xyz="0.06531 0 0.021953" rpy="0 0 0" />
+</xacro:property>
+<xacro:property name="pt_pose" value="${dict(x=-0.02571, z=0.04, pan_z=0.0383)}"/>
+</xacro:if>
+<xacro:unless value="${kit == 'upstream'}">
+<xacro:property name="lidar_joint_pose">
+  <origin xyz="0.0398 0.0001 0.0500" rpy="0 0 1.5708"/>
+</xacro:property>
+<xacro:property name="oak_joint_pose">
+  <origin xyz="0.0684 0 0.0321" rpy="0 0 0" />
+</xacro:property>
+<xacro:property name="pt_pose" value="${dict(x=-0.02001, z=0.0496, pan_z=0.0478)}"/>
+</xacro:unless>
 <xacro:lidar>
 <xacro:insert_block name="lidar_joint_pose" />
@@ -27,10 +47,10 @@
 <xacro:include filename="$(find ugv_description)/urdf/sensors/3d_camera.xacro" />
 <xacro:oak use_gazebo="$(arg use_gazebo)">
-  <origin xyz="0.06531 0 0.021953" rpy="0 0 0" />
+<xacro:insert_block name="oak_joint_pose" />
 </xacro:oak>
 </xacro:unless>
 <xacro:if value="${add_pt}">
 <xacro:include filename="$(find ugv_description)/urdf/sensors/pt.xacro"/>
-<xacro:pt use_gazebo="$(arg use_gazebo)" GZ_VERSION="$(arg GZ_VERSION)" pt_base_link_joint_pose_z="0.04" initial_positions_file="$(find ugv_description)/config/initial_positions.yaml"/>
+<xacro:pt use_gazebo="$(arg use_gazebo)" GZ_VERSION="$(arg GZ_VERSION)" pt_base_link_joint_pose_x="${pt_pose['x']}" pt_base_link_joint_pose_z="${pt_pose['z']}" pan_joint_pose_z="${pt_pose['pan_z']}" initial_positions_file="$(find ugv_description)/config/initial_positions.yaml"/>
 </xacro:if>
 <xacro:if value="${use_gazebo}">

File: src/ugv_main/ugv_description/urdf/sensors/pt.xacro (robot description, xacro)
@@ -1,5 +1,5 @@
 <?xml version="1.0" ?>
 <robot name="pt" xmlns:xacro="http://www.ros.org/wiki/xacro">
-<xacro:macro name="pt" params="use_gazebo GZ_VERSION pt_base_link_joint_pose_z initial_positions_file">
+<xacro:macro name="pt" params="use_gazebo GZ_VERSION pt_base_link_joint_pose_z initial_positions_file pt_base_link_joint_pose_x:=-0.02571 pan_joint_pose_z:=0.0383">
 <xacro:property name="initial_positions" value="${load_yaml(initial_positions_file)['initial_positions']}"/>
 <link name="pt_base_link">
@@ -84,5 +84,5 @@
 </link>
 <joint name="pt_base_link_joint" type="fixed">
-  <origin xyz="-0.02571 0 ${pt_base_link_joint_pose_z}" rpy="0 0 0" />
+  <origin xyz="${pt_base_link_joint_pose_x} 0 ${pt_base_link_joint_pose_z}" rpy="0 0 0" />
   <parent link="base_link" />
   <child link="pt_base_link" />
@@ -90,5 +90,5 @@
 </joint>
 <joint name="pt_base_link_to_pt_link1" type="revolute">
-  <origin xyz="0.0113 0 0.0383" rpy="0 0 0" />
+  <origin xyz="0.0113 0 ${pan_joint_pose_z}" rpy="0 0 0" />
   <parent link="pt_base_link" />
   <child link="pt_link1" />
